Commit message: feat: prepare for updates (#155)

File: aichallenge/workspace/src/aichallenge_submit/racing_kart_description/urdf/vehicle.xacro (robot description, xacro)
@@ -6,5 +6,5 @@
   <link name="base_link">
     <visual>
-      <origin xyz="0 0 0" rpy="0 0 1.57"/>
+      <origin xyz="0.5 0 0" rpy="0 0 1.57"/>
       <geometry>
         <mesh filename="package://racing_kart_description/mesh/kart.dae" scale="1 1 1"/>

File: aichallenge/workspace/src/aichallenge_submit/racing_kart_sensor_kit_description/urdf/sensors.xacro (robot description, xacro)
@@ -14,15 +14,29 @@
     yaw="${calibration['base_link']['sensor_kit_base_link']['yaw']}"
   />
-  <!-- embedded sensors -->
-  <!-- <xacro:include filename="$(find velodyne_description)/urdf/VLP-16.urdf.xacro"/>
-  <xacro:VLP-16 parent="base_link" name="velodyne_rear" topic="velodyne_rear/velodyne_points" hz="10" samples="220" gpu="false">
+  <!-- lidar -->
+  <xacro:include filename="VLP-16.urdf.xacro"/>
+  <xacro:VLP-16
+    name="lidar"
+    parent="base_link">
     <origin
-      xyz="${calibration['base_link']['velodyne_rear_base_link']['x']}
-           ${calibration['base_link']['velodyne_rear_base_link']['y']}
-           ${calibration['base_link']['velodyne_rear_base_link']['z']}"
-      rpy="${calibration['base_link']['velodyne_rear_base_link']['roll']}
-           ${calibration['base_link']['velodyne_rear_base_link']['pitch']}
-           ${calibration['base_link']['velodyne_rear_base_link']['yaw']}"
+      xyz="${calibration['base_link']['lidar_link']['x']}
+           ${calibration['base_link']['lidar_link']['y']}
+           ${calibration['base_link']['lidar_link']['z']}"
+      rpy="${calibration['base_link']['lidar_link']['roll']}
+           ${calibration['base_link']['lidar_link']['pitch']}
+           ${calibration['base_link']['lidar_link']['yaw']}"
     />
-  </xacro:VLP-16> -->
+  </xacro:VLP-16>
+  <!-- camera -->
+  <xacro:include filename="monocular_camera.xacro"/>
+  <xacro:monocular_camera_macro
+    name="camera"
+    parent="base_link"
+    x="${calibration['base_link']['camera_link']['x']}"
+    y="${calibration['base_link']['camera_link']['y']}"
+    z="${calibration['base_link']['camera_link']['z']}"
+    roll="${calibration['base_link']['camera_link']['roll']}"
+    pitch="${calibration['base_link']['camera_link']['pitch']}"
+    yaw="${calibration['base_link']['camera_link']['yaw']}"
+  />
 </robot>
